Commit message: trials with different coordinates

File: test/urdf/robot.urdf (robot description, URDF)
Before this commit: robot robot, 11 links, 10 joints
Joints:
- joint footprint_joint: child base_link -> base_footprint; origin xyz=0.0 0.0 0.05 rpy=0 0 3.14 -> xyz=0.0 0.0 0.05 rpy=0 0 3.1415; parent base_footprint -> base_link
- joint holder3_joint: origin xyz=0.1 -0.1 0.0 rpy=1.5707963267949 0 0.0 -> xyz=0.3 -0.1 0.0 rpy=1.5707963267949 0 0.0
- joint holder4_joint: origin xyz=0.1 0.1 0.0 rpy=1.5707963267949 0 3.14 -> xyz=0.3 0.1 0.0 rpy=1.5707963267949 0 3.14

Commit message: revert previous change

File: test/urdf/robot.urdf (robot description, URDF)
Before this commit: robot robot, 11 links, 10 joints
Joints:
- joint holder3_joint: origin xyz=0.3 -0.1 0.0 rpy=1.5707963267949 0 0.0 -> xyz=0.1 -0.1 0.0 rpy=1.5707963267949 0 0.0
- joint holder4_joint: origin xyz=0.3 0.1 0.0 rpy=1.5707963267949 0 3.14 -> xyz=0.1 0.1 0.0 rpy=1.5707963267949 0 3.14

Commit message: swap axes for wheels (seems to work)

File: test/urdf/robot.urdf (robot description, URDF)
Before this commit: robot robot, 11 links, 10 joints
Joints:
- joint wheel1_joint: axis 1 0 0 -> -1 0 0
- joint wheel2_joint: axis -1 0 0 -> 1 0 0
- joint wheel3_joint: axis 1 0 0 -> -1 0 0
- joint wheel4_joint: axis -1 0 0 -> 1 0 0
